Commit message: Add prismatic vacuum joint for real gripper

File: vgc10_gripper_description/urdf/vgc10_gripper.gazebo.xacro (robot description, xacro)
@@ -1,9 +1,9 @@
 <?xml version="1.0"?>
 <robot xmlns:xacro="http://www.ros.org/wiki/xacro">
-  <xacro:macro name="vacuum_gripper">
+  <xacro:macro name="vacuum_gripper" params="prefix">
    <gazebo>
      <plugin name="gazebo_ros_vacuum_cup_1" filename="libgazebo_ros_vacuum_gripper.so">
        <robotNamespace>/robot</robotNamespace>
-       <bodyName>robot_vgc10_vacuum_cup_1_link</bodyName>
+       <bodyName>${prefix}_gripper_vacuum_cup_1_link</bodyName>
        <topicName>vacuum_cup_1</topicName>
        <serviceNamespace>vacuum_cup_1</serviceNamespace>
@@ -13,5 +13,5 @@
      <plugin name="gazebo_ros_vacuum_cup_2" filename="libgazebo_ros_vacuum_gripper.so">
        <robotNamespace>/robot</robotNamespace>
-       <bodyName>robot_vgc10_vacuum_cup_2_link</bodyName>
+       <bodyName>${prefix}_gripper_vacuum_cup_2_link</bodyName>
        <topicName>vacuum_cup_2</topicName>
        <serviceNamespace>vacuum_cup_2</serviceNamespace>
@@ -21,5 +21,5 @@
      <plugin name="gazebo_ros_vacuum_cup_3" filename="libgazebo_ros_vacuum_gripper.so">
        <robotNamespace>/robot</robotNamespace>
-       <bodyName>robot_vgc10_vacuum_cup_3_link</bodyName>
+       <bodyName>${prefix}_gripper_vacuum_cup_3_link</bodyName>
        <topicName>vacuum_cup_3</topicName>
        <serviceNamespace>vacuum_cup_3</serviceNamespace>
@@ -29,5 +29,5 @@
      <plugin name="gazebo_ros_vacuum_cup_4" filename="libgazebo_ros_vacuum_gripper.so">
        <robotNamespace>/robot</robotNamespace>
-       <bodyName>robot_vgc10_vacuum_cup_4_link</bodyName>
+       <bodyName>${prefix}_gripper_vacuum_cup_4_link</bodyName>
        <topicName>vacuum_cup_4</topicName>
        <serviceNamespace>vacuum_cup_4</serviceNamespace>

File: vgc10_gripper_description/urdf/vgc10_gripper.urdf.xacro (robot description, xacro)
@@ -3,10 +3,10 @@
   <xacro:macro name="vgc10_gripper" params="prefix parent *origin">
     <!--CONTAINER -->
-    <joint name="${prefix}_vgc10_joint" type="fixed">
+    <joint name="${prefix}_base_joint" type="fixed">
 	    <xacro:insert_block name="origin"/>
       <parent link="${parent}"/>
-      <child link="${prefix}_vgc10_link"/>
+      <child link="${prefix}_base_link"/>
     </joint>
-    <link name="${prefix}_vgc10_link">
+    <link name="${prefix}_base_link">
 	    <inertial>
 	      <mass value="0.25"/>
@@ -31,7 +31,21 @@
 	    </collision>
 	  </link>
+    <joint name="${prefix}_vacuum_joint" type="prismatic">
+      <parent link="${prefix}_base_link"/>
+      <child link="${prefix}_vacuum_link" />
+      <origin xyz="0.1042 0 0" rpy="0 0 0" />
+      <limit effort="1000" lower="0.0" upper="0.001" velocity="0.088"/>
+      <axis xyz="1 0 0" />
+    </joint>
+    <link name="${prefix}_vacuum_link">
+        <inertial>
+          <mass value="0.01" />
+          <origin xyz="0 0 0" />
+          <inertia  ixx="1.0" ixy="0.0"  ixz="0.0"  iyy="1.0"  iyz="0.0"  izz="1.0" />
+      </inertial>
+    </link>
     <joint name="${prefix}_vacuum_cup_1_joint" type="revolute">
-      <origin xyz="0.1322 -0.0065 -0.0189" rpy="0 0 0"/>
-      <parent link="${prefix}_vgc10_link"/>
+      <origin xyz="0.028 -0.0065 -0.0189" rpy="0 0 0"/>
+      <parent link="${prefix}_vacuum_link"/>
       <child link="${prefix}_vacuum_cup_1_link"/>
       <axis xyz="1 0 0" rpy="0 0 0" />
@@ -46,6 +60,6 @@
     </link>
     <joint name="${prefix}_vacuum_cup_2_joint" type="revolute">
-      <origin xyz="0.1322 -0.0065 0.0189" rpy="0 0 0"/>
-      <parent link="${prefix}_vgc10_link"/>
+      <origin xyz="0.028 -0.0065 0.0189" rpy="0 0 0"/>
+      <parent link="${prefix}_vacuum_link"/>
       <child link="${prefix}_vacuum_cup_2_link"/>
       <axis xyz="1 0 0" rpy="0 0 0" />
@@ -60,6 +74,6 @@
     </link>
     <joint name="${prefix}_vacuum_cup_3_joint" type="revolute">
-      <origin xyz="0.1322 0.02 0" rpy="0 0 0"/>
-      <parent link="${prefix}_vgc10_link"/>
+      <origin xyz="0.028 0.02 0" rpy="0 0 0"/>
+      <parent link="${prefix}_vacuum_link"/>
       <child link="${prefix}_vacuum_cup_3_link"/>
       <limit effort="30" velocity="1.0" lower="-0.1" upper="0.1" />
@@ -74,6 +88,6 @@
     </link>
     <joint name="${prefix}_vacuum_cup_4_joint" type="revolute">
-      <origin xyz="0.1322 0 0" rpy="0 0 0"/>
-      <parent link="${prefix}_vgc10_link"/>
+      <origin xyz="0.028 0 0" rpy="0 0 0"/>
+      <parent link="${prefix}_vacuum_link"/>
       <child link="${prefix}_vacuum_cup_4_link"/>
       <limit effort="30" velocity="1.0" lower="-0.1" upper="0.1" />
@@ -88,4 +102,13 @@
     </link>
     <!-- Transmission -->
+    <transmission name="${prefix}_vacuum_transmission"  type="SimpleTransmission">
+      <type>transmission_interface/SimpleTransmission</type>
+      <actuator name="${prefix}_vacuum_joint_motor">
+          <mechanicalReduction>1</mechanicalReduction>
+      </actuator>
+      <joint name="${prefix}_vacuum_joint">
+          <hardwareInterface>hardware_interface/PositionJointInterface</hardwareInterface>
+      </joint>
+    </transmission>
     <transmission name="${prefix}_vacuum_cup_1_joint_transmission">
       <type>transmission_interface/SimpleTransmission</type>
